File: hardware/Serial-7-Segment-Display.brd (EAGLE design)
At the start: 40.6 x 22.9 mm, 30 parts

Commit message: fixed some comments, re-worked pin labels in sch.
Fixed comments in System_Functions.ino which mapped Arduino pins to
display pins
Some labels on the schematic did not match the display pin they
connected to. Renamed those nets to make more sense.
Added a pdf of current schematic, not sure if this'll be sustainable.
Trying it out.
Defaulted display type to S7S in the firmware.
Connections:
- net A/COL renamed C/COL
- net F renamed F/APOS
- net G/APOS renamed G
- removed net C: ATMEGA328P-AU.23, R4.2
- new net A: ATMEGA328P-AU.12, R3.2
- net B: now also ATMEGA328P-AU.23, R4.2; no longer ATMEGA328P-AU.12, R3.2
Routing:
- net C: track 29.3 -> 0.00 mm, vias 2 -> 0
- net B: track 14.3 -> 29.3 mm
- net A: track 0.00 -> 14.3 mm, vias 0 -> 2
Changed lines of the file:
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@@
 <?xml version="1.0" encoding="utf-8"?>
 <!DOCTYPE eagle SYSTEM "eagle.dtd">
-<eagle version="6.1">
+<eagle version="6.4">
 <drawing>
 <settings>
@@
 </class>
 </classes>
-<designrules>
+<designrules name="default">
 <description language="en">&lt;b&gt;EAGLE Design Rules&lt;/b&gt;
 &lt;p&gt;
@@
 <wire x1="9.017" y1="3.556" x2="7.747" y2="4.826" width="0.254" layer="1"/>
 </signal>
-<signal name="G/APOS">
+<signal name="G">
 <contactref element="R9" pad="2"/>
 <contactref element="ATMEGA328P-AU" pad="9"/>
@@
 <wire x1="12.635225" y1="12.485425" x2="13.1038" y2="12.954" width="0.254" layer="1"/>
 </signal>
-<signal name="F">
+<signal name="F/APOS">
 <contactref element="R8" pad="2"/>
 <contactref element="ATMEGA328P-AU" pad="11"/>
@@
 <wire x1="1.905" y1="11.176" x2="1.905" y2="10.795" width="0.254" layer="16"/>
 </signal>
-<signal name="C">
+<signal name="B">
 <contactref element="R4" pad="2"/>
 <contactref element="ATMEGA328P-AU" pad="23"/>
@@
 <wire x1="4.156571875" y1="12.065" x2="4.156571875" y2="11.303" width="0.254" layer="1"/>
 </signal>
-<signal name="B">
+<signal name="A">
 <contactref element="R3" pad="2"/>
 <contactref element="ATMEGA328P-AU" pad="12"/>
@@
 <wire x1="10.5986875" y1="13.843" x2="20.828" y2="13.843" width="0.254" layer="16"/>
 </signal>
-<signal name="A/COL">
+<signal name="C/COL">
 <contactref element="R2" pad="2"/>
 <contactref element="ATMEGA328P-AU" pad="10"/>
