File: hardware/Serial-7-Segment-Display.sch (EAGLE design)
At the start: 29 parts

Commit message: fixed some comments, re-worked pin labels in sch.
Fixed comments in System_Functions.ino which mapped Arduino pins to
display pins
Some labels on the schematic did not match the display pin they
connected to. Renamed those nets to make more sense.
Added a pdf of current schematic, not sure if this'll be sustainable.
Trying it out.
Defaulted display type to S7S in the firmware.
Connections:
- net A/COL renamed C/COL
- net F renamed F/APOS
- net G/APOS renamed G
- removed net C: ATMEGA328P-AU.PC0(ADC0), R4.2
- new net A: ATMEGA328P-AU.PB0(ICP), R3.2
- net B: now also ATMEGA328P-AU.PC0(ADC0), R4.2; no longer ATMEGA328P-AU.PB0(ICP), R3.2
Changed lines of the file:
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@@
 <?xml version="1.0" encoding="utf-8"?>
 <!DOCTYPE eagle SYSTEM "eagle.dtd">
-<eagle version="6.1">
+<eagle version="6.4">
 <drawing>
 <settings>
@@
 </segment>
 </net>
-<net name="G/APOS" class="0">
+<net name="G" class="0">
 <segment>
 <pinref part="R9" gate="G$1" pin="2"/>
@@
 </segment>
 </net>
-<net name="F" class="0">
+<net name="F/APOS" class="0">
 <segment>
 <pinref part="R8" gate="G$1" pin="2"/>
@@
 </segment>
 </net>
-<net name="C" class="0">
+<net name="B" class="0">
 <segment>
 <pinref part="R4" gate="G$1" pin="2"/>
@@
 </segment>
 </net>
-<net name="B" class="0">
+<net name="A" class="0">
 <segment>
 <pinref part="R3" gate="G$1" pin="2"/>
@@
 </segment>
 </net>
-<net name="A/COL" class="0">
+<net name="C/COL" class="0">
 <segment>
 <pinref part="R2" gate="G$1" pin="2"/>
